File: imu.kicad_sch (KiCad schematic)
At the start: 1 part, among them U4 LSM6DSM

Commit message: first commit
Parts:
- renumbered U4 to U601
Changed lines of the file:
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@@
 		(dnp no)
 		(fields_autoplaced yes)
-		(property "Reference" "U4"
+		(property "Reference" "U601"
 			(at 135.4933 91.44 0)
 			(show_name no)
@@
 			(project "watt_city_car_pcb"
 				(path "/72ee6c6c-9225-4cd9-b8d3-156d5f3d5230/d81bad0f-b8dc-4a6a-8f5b-8ea64f0dd5bb"
-					(reference "U4")
+					(reference "U601")
 					(unit 1)
 				)
