File: laserSensor.kicad_sch (KiCad schematic)
At the start: 1 part, among them U6 VL53L0CXV0DH/1

Commit message: first commit
Parts:
- renumbered U6 to U701
Changed lines of the file:
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@@
 		(dnp no)
 		(fields_autoplaced yes)
-		(property "Reference" "U6"
+		(property "Reference" "U701"
 			(at 134.62 86.36 0)
 			(show_name no)
@@
 			(project "watt_city_car_pcb"
 				(path "/72ee6c6c-9225-4cd9-b8d3-156d5f3d5230/4e145819-59fd-45dd-a08f-edddbdb0b5d2"
-					(reference "U6")
+					(reference "U701")
 					(unit 1)
 				)
