File: usb.kicad_sch (KiCad schematic)
At the start: 5 parts, among them J1 USB_C_Receptacle_USB2.0_14P, U2 SLLC23T5V2U

Commit message: added sensor sheets
Connections:
- net +5V_USB: now also D1001.2 (A); no longer D1001.1 (K)
- net at J1.A4 (VBUS), J1.A9 (VBUS), J1.B4 (VBUS)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: now also D1001.1 (K); no longer D1001.2 (A)
Other:
- moved on the sheet: D1001
Changed lines of the file:
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@@
 	(symbol
 		(lib_id "bfr_diodes:1N5819WS")
-		(at 138.43 83.82 180)
+		(at 138.43 83.82 0)
 		(unit 1)
 		(body_style 1)
@@
 		(fields_autoplaced yes)
 		(property "Reference" "D1001"
-			(at 138.7475 90.17 0)
+			(at 138.1125 77.47 0)
 			(show_name no)
 			(do_not_autoplace no)
@@
 		)
 		(property "Value" "600m"
-			(at 138.7475 87.63 0)
+			(at 138.1125 80.01 0)
 			(show_name no)
 			(do_not_autoplace no)
@@
 		)
 		(property "Footprint" "Diode_SMD:D_SOD-323_HandSoldering"
-			(at 138.43 87.63 0)
+			(at 138.43 80.01 0)
 			(hide yes)
 			(show_name no)
@@
 		)
 		(property "Datasheet" "https://wmsc.lcsc.com/wmsc/upload/file/pdf/v2/lcsc/2204281430_Guangdong-Hottech-1N5819WS_C191023.pdf"
-			(at 138.43 87.63 0)
+			(at 138.43 80.01 0)
 			(hide yes)
 			(show_name no)
@@
 		)
 		(property "Description" "1A 600mV SOD-323 Schottky Diode"
-			(at 138.43 87.63 0)
+			(at 138.43 80.01 0)
 			(hide yes)
 			(show_name no)
@@
 		)
 		(property "LCSC P/N" "C191023"
-			(at 138.684 87.63 0)
+			(at 138.176 80.01 0)
 			(hide yes)
 			(show_name no)
@@
 		)
 		(property "Digikey P/N" "5272-B5819WSCT-ND"
-			(at 138.43 87.63 0)
+			(at 138.43 80.01 0)
 			(hide yes)
 			(show_name no)
@@
 		)
 		(property "Mouser P/N" "833-B5819WS-TP"
-			(at 138.684 87.63 0)
+			(at 138.176 80.01 0)
 			(hide yes)
 			(show_name no)
@@
 		)
 		(property "Order From" "Digikey"
-			(at 138.43 87.884 0)
+			(at 138.43 79.756 0)
 			(hide yes)
 			(show_name no)
@@
 		)
 		(property "JLCPCB Basic Part" "Yes"
-			(at 138.43 87.63 0)
+			(at 138.43 80.01 0)
 			(hide yes)
 			(show_name no)
@@
 		)
 		(property "Pretty Name" "1A SOD-323 Schottky Diode"
-			(at 138.43 87.63 0)
+			(at 138.43 80.01 0)
 			(hide yes)
 			(show_name no)
@@
 		)
 		(property "Sim.Library" "${BFRUH_DIR}\\Electronics\\spice_models\\bfr_diodes\\1N5819WS.lib"
-			(at 138.43 87.63 0)
+			(at 138.43 80.01 0)
 			(hide yes)
 			(show_name no)
@@
 		)
 		(property "Sim.Name" "1N5819WS"
-			(at 138.684 87.63 0)
+			(at 138.176 80.01 0)
 			(hide yes)
 			(show_name no)
@@
 		)
 		(property "Sim.Device" "SUBCKT"
-			(at 138.43 87.63 0)
+			(at 138.43 80.01 0)
 			(hide yes)
 			(show_name no)
@@
 		)
 		(property "Sim.Pins" "1=K 2=A"
-			(at 138.684 87.63 0)
+			(at 138.176 80.01 0)
 			(hide yes)
 			(show_name no)
@@
 		)
 		(property "Created by" "Manual Entry"
-			(at 138.43 87.63 0)
-			(hide yes)
-			(show_name no)
+			(at 138.43 80.01 0)
+			(hide yes)
+			(show_name no)

Commit message: first commit
Parts:
- renumbered D1001 to D501, J1 to J501, R2 to R501, R1 to R502, U2 to U501
Connections:
- net +5V_USB: now also D501.1 (K); no longer D501.2 (A)
- net at J501.A4 (VBUS), J501.A9 (VBUS), J501.B4 (VBUS)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: now also D501.2 (A); no longer D501.1 (K)
Other:
- moved on the sheet: D501
Changed lines of the file:
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@@
 	)
 	(hierarchical_label "+5V_USB"
-		(shape input)
+		(shape output)
 		(at 144.78 83.82 0)
 		(effects
@@
 		(dnp no)
 		(fields_autoplaced yes)
-		(property "Reference" "J1"
+		(property "Reference" "J501"
 			(at 99.06 76.2 0)
 			(show_name no)
@@
 			(project "watt_city_car_pcb"
 				(path "/72ee6c6c-9225-4cd9-b8d3-156d5f3d5230/59e3dad0-55dc-4a04-87f2-2c349902244d/b5be7689-98d6-47fe-8b13-538f7b8d313e"
-					(reference "J1")
+					(reference "J501")
 					(unit 1)
 				)
@@
 		(in_pos_files yes)
 		(dnp no)
-		(property "Reference" "R2"
+		(property "Reference" "R501"
 			(at 113.284 117.602 90)
 			(show_name no)
@@
 			(project "watt_city_car_pcb"
 				(path "/72ee6c6c-9225-4cd9-b8d3-156d5f3d5230/59e3dad0-55dc-4a04-87f2-2c349902244d/b5be7689-98d6-47fe-8b13-538f7b8d313e"
-					(reference "R2")
+					(reference "R501")
 					(unit 1)
 				)
@@
 		(dnp no)
 		(fields_autoplaced yes)
-		(property "Reference" "#PWR02"
+		(property "Reference" "#PWR0501"
 			(at 99.06 132.08 0)
 			(hide yes)
@@
 			(project "watt_city_car_pcb"
 				(path "/72ee6c6c-9225-4cd9-b8d3-156d5f3d5230/59e3dad0-55dc-4a04-87f2-2c349902244d/b5be7689-98d6-47fe-8b13-538f7b8d313e"
-					(reference "#PWR02")
+					(reference "#PWR0501")
 					(unit 1)
 				)
@@
 		(dnp no)
 		(fields_autoplaced yes)
-		(property "Reference" "U2"
+		(property "Reference" "U501"
 			(at 154.94 112.5854 0)
 			(show_name no)
@@
 			(project "watt_city_car_pcb"
 				(path "/72ee6c6c-9225-4cd9-b8d3-156d5f3d5230/59e3dad0-55dc-4a04-87f2-2c349902244d/b5be7689-98d6-47fe-8b13-538f7b8d313e"
-					(reference "U2")
+					(reference "U501")
 					(unit 1)
 				)
@@
 		(dnp no)
 		(fields_autoplaced yes)
-		(property "Reference" "#PWR07"
+		(property "Reference" "#PWR0502"
 			(at 148.59 128.27 0)
 			(hide yes)
@@
 			(project "watt_city_car_pcb"
 				(path "/72ee6c6c-9225-4cd9-b8d3-156d5f3d5230/59e3dad0-55dc-4a04-87f2-2c349902244d/b5be7689-98d6-47fe-8b13-538f7b8d313e"
-					(reference "#PWR07")
+					(reference "#PWR0502")
 					(unit 1)
 				)
@@
 	(symbol
 		(lib_id "bfr_diodes:1N5819WS")
-		(at 138.43 83.82 0)
+		(at 138.43 83.82 180)
 		(unit 1)
 		(body_style 1)
@@
 		(dnp no)
 		(fields_autoplaced yes)
-		(property "Reference" "D1001"
-			(at 138.1125 77.47 0)
+		(property "Reference" "D501"
+			(at 138.7475 77.47 0)
 			(show_name no)
 			(do_not_autoplace no)
@@
 		)
 		(property "Value" "600m"
-			(at 138.1125 80.01 0)
+			(at 138.7475 80.01 0)
 			(show_name no)
 			(do_not_autoplace no)
@@
 		)
 		(property "Footprint" "Diode_SMD:D_SOD-323_HandSoldering"
-			(at 138.43 80.01 0)
+			(at 138.43 87.63 0)
 			(hide yes)
 			(show_name no)
@@
 		)
 		(property "Datasheet" "https://wmsc.lcsc.com/wmsc/upload/file/pdf/v2/lcsc/2204281430_Guangdong-Hottech-1N5819WS_C191023.pdf"
-			(at 138.43 80.01 0)
+			(at 138.43 87.63 0)
 			(hide yes)
 			(show_name no)
@@
 		)
 		(property "Description" "1A 600mV SOD-323 Schottky Diode"
-			(at 138.43 80.01 0)
+			(at 138.43 87.63 0)
 			(hide yes)
 			(show_name no)
@@
 		)
 		(property "LCSC P/N" "C191023"
-			(at 138.176 80.01 0)
+			(at 138.684 87.63 0)
 			(hide yes)
 			(show_name no)
@@
 		)
 		(property "Digikey P/N" "5272-B5819WSCT-ND"
-			(at 138.43 80.01 0)
+			(at 138.43 87.63 0)
 			(hide yes)
 			(show_name no)
@@
 		)
 		(property "Mouser P/N" "833-B5819WS-TP"
-			(at 138.176 80.01 0)
+			(at 138.684 87.63 0)
 			(hide yes)
 			(show_name no)
@@
 		)
 		(property "Order From" "Digikey"
-			(at 138.43 79.756 0)
+			(at 138.43 87.884 0)
 			(hide yes)
 			(show_name no)
@@
 		)
 		(property "JLCPCB Basic Part" "Yes"
-			(at 138.43 80.01 0)
+			(at 138.43 87.63 0)
 			(hide yes)
 			(show_name no)
@@
 		)
 		(property "Pretty Name" "1A SOD-323 Schottky Diode"
-			(at 138.43 80.01 0)
+			(at 138.43 87.63 0)
 			(hide yes)
 			(show_name no)
@@
 		)
 		(property "Sim.Library" "${BFRUH_DIR}\\Electronics\\spice_models\\bfr_diodes\\1N5819WS.lib"
-			(at 138.43 80.01 0)
+			(at 138.43 87.63 0)
 			(hide yes)
 			(show_name no)
@@
 		)
 		(property "Sim.Name" "1N5819WS"
-			(at 138.176 80.01 0)
+			(at 138.684 87.63 0)
 			(hide yes)
 			(show_name no)
@@
 		)
 		(property "Sim.Device" "SUBCKT"
-			(at 138.43 80.01 0)
+			(at 138.43 87.63 0)
 			(hide yes)
 			(show_name no)
@@
 		)
 		(property "Sim.Pins" "1=K 2=A"
-			(at 138.176 80.01 0)
+			(at 138.684 87.63 0)
 			(hide yes)
 			(show_name no)
@@
 		)
 		(property "Created by" "Manual Entry"
-			(at 138.43 80.01 0)
+			(at 138.43 87.63 0)
 			(hide yes)
 			(show_name no)
@@
 			(project "watt_city_car_pcb"
 				(path "/72ee6c6c-9225-4cd9-b8d3-156d5f3d5230/59e3dad0-55dc-4a04-87f2-2c349902244d/b5be7689-98d6-47fe-8b13-538f7b8d313e"
-					(reference "D1001")
+					(reference "D501")
 					(unit 1)
 				)
@@
 		(in_pos_files yes)
 		(dnp no)
-		(property "Reference" "R1"
+		(property "Reference" "R502"
 			(at 126.492 114.554 90)
 			(show_name no)
@@
 			(project "watt_city_car_pcb"
 				(path "/72ee6c6c-9225-4cd9-b8d3-156d5f3d5230/59e3dad0-55dc-4a04-87f2-2c349902244d/b5be7689-98d6-47fe-8b13-538f7b8d313e"
-					(reference "R1")
+					(reference "R502")
 					(unit 1)
 				)
