File: power.kicad_sch (KiCad schematic)
At the start: 2 parts, among them J2 Conn_01x01_Socket, J3 Conn_01x01_Socket

Commit message: added sensor sheets
Other:
- sheet ldo ports: added 3V3; removed none
Changed lines of the file:
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@@
+		)
+	)
+	(bus
+		(pts
+			(xy 104.14 140.97) (xy 130.81 140.97)
+		)
+		(stroke
+			(width 0)
+			(type default)
+		)
+	)
+	(wire
+		(pts
+			(xy 179.07 134.62) (xy 185.42 134.62)
+		)
+		(stroke
+			(width 0)
+			(type default)
 		)
 	)
@@
 		)
 	)
+	(wire
+		(pts
+			(xy 176.53 127) (xy 185.42 127)
+		)
+		(stroke
+			(width 0)
+			(type default)
+		)
+	)
+	(label "{USB_D+, USB_D-}"
+		(at 106.68 140.97 0)
+		(effects
+			(font
+				(size 1.27 1.27)
+			)
+			(justify left bottom)
+		)
+	)
+	(hierarchical_label "3V3"
+		(shape input)
+		(at 179.07 134.62 180)
+		(effects
+			(font
+				(size 1.27 1.27)
+			)
+			(justify right)
+		)
+	)
 	(hierarchical_label "VBATT"
-		(shape output)
+		(shape input)
 		(at 124.46 91.44 180)
 		(effects
@@
 			)
 			(justify right)
+		)
+	)
+	(hierarchical_label "VBATT"
+		(shape input)
+		(at 176.53 127 180)
+		(effects
+			(font
+				(size 1.27 1.27)
+			)
+			(justify right)
+		)
+	)
+	(hierarchical_label "USB"
+		(shape input)
+		(at 130.81 140.97 0)
+		(effects
+			(font
+				(size 1.27 1.27)
+			)
+			(justify left)
 		)
 	)
@@
 			(effects
 				(font
+					(size 1.27 1.27)
+				)
+				(justify left)
+			)
+		)
+		(pin "3V3" input
+			(at 185.42 134.62 180)
+			(effects
+				(font

Commit message: first commit
Parts:
- renumbered J2 to J301, J3 to J302
Changed lines of the file:
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@@
 		(dnp no)
 		(fields_autoplaced yes)
-		(property "Reference" "J3"
+		(property "Reference" "J302"
 			(at 135.89 102.8699 0)
 			(show_name no)
@@
 			(project "watt_city_car_pcb"
 				(path "/72ee6c6c-9225-4cd9-b8d3-156d5f3d5230/59e3dad0-55dc-4a04-87f2-2c349902244d"
-					(reference "J3")
+					(reference "J302")
 					(unit 1)
 				)
@@
 		(dnp no)
 		(fields_autoplaced yes)
-		(property "Reference" "J2"
+		(property "Reference" "J301"
 			(at 135.89 90.1699 0)
 			(show_name no)
@@
 			(project "watt_city_car_pcb"
 				(path "/72ee6c6c-9225-4cd9-b8d3-156d5f3d5230/59e3dad0-55dc-4a04-87f2-2c349902244d"
-					(reference "J2")
+					(reference "J301")
 					(unit 1)
 				)
@@
 		(dnp no)
 		(fields_autoplaced yes)
-		(property "Reference" "#PWR05"
+		(property "Reference" "#PWR0301"
 			(at 123.19 110.49 0)
 			(hide yes)
@@
 			(project "watt_city_car_pcb"
 				(path "/72ee6c6c-9225-4cd9-b8d3-156d5f3d5230/59e3dad0-55dc-4a04-87f2-2c349902244d"
-					(reference "#PWR05")
+					(reference "#PWR0301")
 					(unit 1)
 				)
@@
 			)
 		)
-		(pin "+5V_USB" input
+		(pin "+5V_USB" output
 			(at 104.14 130.81 0)
 			(effects

Commit message: preliminary schematic
Other:
- sheet ldo ports: added +5V_USB; removed 3V3
Changed lines of the file:
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@@
 	(wire
 		(pts
-			(xy 124.46 91.44) (xy 129.54 91.44)
+			(xy 121.92 91.44) (xy 129.54 91.44)
 		)
 		(stroke
@@
 	(bus
 		(pts
-			(xy 104.14 140.97) (xy 130.81 140.97)
+			(xy 104.14 138.43) (xy 130.81 138.43)
 		)
 		(stroke
@@
 	(wire
 		(pts
-			(xy 179.07 134.62) (xy 185.42 134.62)
+			(xy 104.14 128.27) (xy 147.32 128.27)
 		)
 		(stroke
@@
 	(wire
 		(pts
-			(xy 176.53 127) (xy 185.42 127)
+			(xy 138.43 124.46) (xy 147.32 124.46)
 		)
 		(stroke
@@
 		)
 	)
-	(label "{USB_D+, USB_D-}"
-		(at 106.68 140.97 0)
+	(label "VBATT"
+		(at 138.43 124.46 0)
 		(effects
 			(font
@@
 		)
 	)
-	(hierarchical_label "3V3"
-		(shape input)
-		(at 179.07 134.62 180)
+	(label "{USB_D+, USB_D-}"
+		(at 106.68 138.43 0)
 		(effects
 			(font
 				(size 1.27 1.27)
 			)
-			(justify right)
-		)
-	)
-	(hierarchical_label "VBATT"
-		(shape input)
-		(at 124.46 91.44 180)
+			(justify left bottom)
+		)
+	)
+	(label "VBATT"
+		(at 121.92 91.44 0)
 		(effects
 			(font
 				(size 1.27 1.27)
 			)
-			(justify right)
-		)
-	)
-	(hierarchical_label "VBATT"
-		(shape input)
-		(at 176.53 127 180)
-		(effects
-			(font
-				(size 1.27 1.27)
-			)
-			(justify right)
+			(justify left bottom)
 		)
 	)
 	(hierarchical_label "USB"
-		(shape input)
-		(at 130.81 140.97 0)
+		(shape bidirectional)
+		(at 130.81 138.43 0)
 		(effects
 			(font
@@
 	)
 	(sheet
-		(at 185.42 121.92)
+		(at 147.32 119.38)
 		(size 34.29 19.05)
 		(exclude_from_sim no)
@@
 		)
 		(property "Sheetname" "ldo"
-			(at 185.42 121.2084 0)
+			(at 147.32 118.6684 0)
 			(show_name no)
 			(do_not_autoplace no)
@@
 		)
 		(property "Sheetfile" "ldo.kicad_sch"
-			(at 185.42 141.5546 0)
+			(at 147.32 139.0146 0)
 			(show_name no)
 			(do_not_autoplace no)
@@
 		)
 		(property "Field2" ""
-			(at 185.42 121.92 0)
+			(at 147.32 119.38 0)
 			(hide yes)
 			(show_name no)
@@
 		)
 		(pin "VBATT" input
-			(at 185.42 127 180)
-			(effects
-				(font
-					(size 1.27 1.27)
-				)
-				(justify left)
-			)
-		)
-		(pin "3V3" input
-			(at 185.42 134.62 180)
+			(at 147.32 124.46 180)
+			(effects
+				(font
+					(size 1.27 1.27)
+				)
+				(justify left)
+			)
+		)
+		(pin "+5V_USB" input
+			(at 147.32 128.27 180)
 			(effects
 				(font
@@
 	)
 	(sheet
-		(at 59.69 121.92)
+		(at 59.69 119.38)
 		(size 44.45 26.67)
 		(exclude_from_sim no)
@@
 		)
 		(property "Sheetname" "usb"
-			(at 59.69 121.2084 0)
+			(at 59.69 118.6684 0)
 			(show_name no)
 			(do_not_autoplace no)
@@
 		)
 		(property "Sheetfile" "usb.kicad_sch"
-			(at 59.69 149.1746 0)
+			(at 59.69 146.6346 0)
 			(show_name no)
 			(do_not_autoplace no)
@@
 		)
 		(pin "+5V_USB" output
-			(at 104.14 130.81 0)
+			(at 104.14 128.27 0)
 			(effects
 				(font
@@
 			)
 		)
-		(pin "USB" input
-			(at 104.14 140.97 0)
-			(effects
-				(font
+		(pin "USB" bidirectional
+			(at 104.14 138.43 0)
+			(effects
+				(font
