File: watt_city_car_pcb.kicad_sch (KiCad schematic)
At the start: 0 parts

Commit message: added sensor sheets
Other:
- added sheet imu (imu.kicad_sch)
- added sheet laserSensor (laserSensor.kicad_sch)
- sheet microcontroller ports: added 3V3, USB; removed none
- sheet power ports: added 3V3, USB; removed none
Changed lines of the file:
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@@
+		)
+	)
+	(bus
+		(pts
+			(xy 71.12 101.6) (xy 85.09 101.6)
+		)
+		(stroke
+			(width 0)
+			(type default)
+		)
+	)
+	(bus
+		(pts
+			(xy 85.09 101.6) (xy 85.09 99.06)
+		)
+		(stroke
+			(width 0)
+			(type default)
+		)
+	)
+	(bus
+		(pts
+			(xy 85.09 99.06) (xy 87.63 99.06)
+		)
+		(stroke
+			(width 0)
+			(type default)
+		)
+	)
+	(wire
+		(pts
+			(xy 71.12 90.17) (xy 87.63 90.17)
+		)
+		(stroke
+			(width 0)
+			(type default)
+		)
+	)
+	(sheet
+		(at 154.94 123.19)
+		(size 24.13 16.51)
+		(exclude_from_sim no)
+		(in_bom yes)
+		(on_board yes)
+		(dnp no)
+		(fields_autoplaced yes)
+		(stroke
+			(width 0.1524)
+			(type solid)
+		)
+		(fill
+			(color 0 0 0 0)
+		)
+		(property "Sheetname" "laserSensor"
+			(at 154.94 122.4784 0)
+			(show_name no)
+			(do_not_autoplace no)
+			(effects
+				(font
+					(size 1.27 1.27)
+				)
+				(justify left bottom)
+			)
+		)
+		(property "Sheetfile" "laserSensor.kicad_sch"
+			(at 154.94 140.2846 0)
+			(show_name no)
+			(do_not_autoplace no)
+			(effects
+				(font
+					(size 1.27 1.27)
+				)
+				(justify left top)
+			)
+		)
+		(instances
+			(project "watt_city_car_pcb"
+				(path "/72ee6c6c-9225-4cd9-b8d3-156d5f3d5230"
+					(page "7")
+				)
+			)
 		)
 	)
@@
 			)
 		)
-		(pin "VBATT" output
-			(at 71.12 93.98 0)
+		(pin "3V3" input
+			(at 71.12 90.17 0)
 			(effects
 				(font
@@
 			)
 		)
+		(pin "VBATT" input
+			(at 71.12 97.79 0)
+			(effects
+				(font
+					(size 1.27 1.27)
+				)
+				(justify right)
+			)
+		)
+		(pin "USB" input
+			(at 71.12 101.6 0)
+			(effects
+				(font
+					(size 1.27 1.27)
+				)
+				(justify right)
+			)
+		)
 		(instances
 			(project "watt_city_car_pcb"
@@
 	)
 	(sheet
-		(at 97.79 77.47)
+		(at 87.63 81.28)
 		(size 29.21 22.86)
 		(exclude_from_sim no)
@@
 		)
 		(property "Sheetname" "microcontroller"
-			(at 97.79 76.7584 0)
+			(at 87.63 80.5684 0)
 			(show_name no)
 			(do_not_autoplace no)
@@
 		)
 		(property "Sheetfile" "microcontroller.kicad_sch"
-			(at 97.79 100.9146 0)
-			(show_name no)
-			(do_not_autoplace no)
-			(effects
-				(font
-					(size 1.27 1.27)
-				)
-				(justify left top)
+			(at 87.63 104.7246 0)
+			(show_name no)
+			(do_not_autoplace no)
+			(effects
+				(font
+					(size 1.27 1.27)
+				)
+				(justify left top)
+			)
+		)
+		(pin "3V3" input
+			(at 87.63 90.17 180)
+			(effects
+				(font
+					(size 1.27 1.27)
+				)
+				(justify left)
+			)
+		)
+		(pin "USB" input
+			(at 87.63 99.06 180)
+			(effects
+				(font
+					(size 1.27 1.27)
+				)
+				(justify left)
 			)
 		)
@@
 				)
 			)
+		)
+	)
+	(sheet
+		(at 152.4 92.71)
+		(size 27.94 19.05)
+		(exclude_from_sim no)
+		(in_bom yes)
+		(on_board yes)
+		(dnp no)
+		(fields_autoplaced yes)
+		(stroke
+			(width 0.1524)
+			(type solid)
+		)
+		(fill
+			(color 0 0 0 0)
+		)
+		(property "Sheetname" "imu"
+			(at 152.4 91.9984 0)
+			(show_name no)
+			(do_not_autoplace no)
+			(effects
+				(font
+					(size 1.27 1.27)
+				)
+				(justify left bottom)
+			)
+		)
+		(property "Sheetfile" "imu.kicad_sch"
+			(at 152.4 112.3446 0)
+			(show_name no)
+			(do_not_autoplace no)
+			(effects
+				(font
+					(size 1.27 1.27)
+				)
+				(justify left top)
+			)
+		)
+		(instances
+			(project "watt_city_car_pcb"
+				(path "/72ee6c6c-9225-4cd9-b8d3-156d5f3d5230"
+					(page "6")
+				)
+			)

Commit message: preliminary schematic
Other:
- removed sheet laserSensor
- added sheet distSensor (distSensor.kicad_sch)
- sheet imu ports: added IMU_INT1, IMU_INT2, IMU_SPI; removed none
- sheet microcontroller ports: added IMU_INT1, IMU_INT2, IMU_SPI, LASER_I2C, laser0_interrupt, laser0_xshut, laser1_interrupt, laser1_xshut, laser2_interrupt, laser2_xshut; removed 3V3
- sheet power ports: added none; removed 3V3, VBATT
