File: hardware/distSensor.kicad_sch (KiCad schematic)
At the start: 2 parts, among them J301 Conn_01x01_Socket, J302 Conn_01x01_Socket

Commit message: updated pcb
Parts:
- removed J301, J302: Conn_01x01_Socket, symbol Connector:Conn_01x01_Socket
- added J4: J_VL53L0X, Connector_PinHeader_2.54mm:PinHeader_1x06_P2.54mm_Horizontal, symbol Connector_Generic:Conn_01x06
Connections:
- net GND: now also J4.2 (Pin_2)
- new net +3.3V: J4.1 (Pin_1)
- new net LASER_I2C.LASER_I2C_SCL: J4.3 (Pin_3)
- new net LASER_I2C.LASER_I2C_SDA: J4.4 (Pin_4)
- new net laser0_interrupt: J4.6 (Pin_6)
- new net laser0_xshut: J4.5 (Pin_5)
Other:
- removed sheet ldo
- removed sheet powerProtection
- removed sheet usb
- note added: "interrupt is input_pullup xshut is output"
