File: hardware/laserSensor.kicad_sch (KiCad schematic)
At the start: 1 part, among them U701 VL53L0CXV0DH/1

Commit message: updated pcb
Parts:
- added C701: 100n, Capacitor_SMD:C_0603_1608Metric_Pad1.08x0.95mm_HandSolder, symbol bfr_capacitors:06035C104KAT2A
- added C702: 4.7u, Capacitor_SMD:C_0805_2012Metric_Pad1.18x1.45mm_HandSolder, symbol bfr_capacitors:KGM21AR51A475KU
- added R701, R703: 4.7k, Resistor_SMD:R_0805_2012Metric_Pad1.20x1.40mm_HandSolder, symbol bfr_master:RMCF0805FT4K70
- added R702, R704: 10k, Resistor_SMD:R_0603_1608Metric_Pad0.98x0.95mm_HandSolder, symbol bfr_resistors:RMCF0603FT10K0
Connections:
- net +3.3V: now reaches U701.1 (AVDDVCSEL)
- net +3.3V: now also U701.11 (AVDD), C701.1, C702.1, R701.2, R702.1, R703.2, R704.2
- net at U701.10 (SCL): now also R701.1
- net GND: now reaches U701.12 (GND4)
- net GND: now also U701.2 (AVSSVCSEL), U701.3 (GND), U701.4 (GND2), U701.6 (GND3), C701.2, C702.2
- net at U701.5 (XSHUT): now also R702.2
- net laser_interrupt: now reaches U701.7 (GPIO1)
- net laser_interrupt: now also R704.1
- net at U701.9 (SDA): now also R703.1
