File: hardware/usb.kicad_sch (KiCad schematic)
At the start: 5 parts, among them J501 USB_C_Receptacle_USB2.0_14P, U501 SLLC23T5V2U

Commit message: updated pcb
Changed lines of the file:
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@@
 	)
 	(hierarchical_label "USB"
-		(shape input)
+		(shape bidirectional)
 		(at 184.15 97.79 0)
 		(effects
